Commit message: Added lidar - need to test in rtabmap

File: lunabot_sim/dummy_bot_description/urdf/dummy_bot.xacro (robot description, xacro)
@@ -9,4 +9,7 @@
 <xacro:property name="wheelRadius" value="0.2"/>
 <xacro:property name="wheelMass" value="5"/>
+<xacro:property name="lidarMass" value="0.190" />
+<xacro:property name="lidarRadius" value="0.038" />
+<xacro:property name="lidarHeight" value="0.041" />
 <xacro:macro name="box_inertia" params="m x y z">
   <inertia  ixx="${m*(y*y+z*z)/12}" ixy = "0" ixz = "0"
@@ -124,4 +127,25 @@
   </collision>
 </link>
+<link name="lidar">
+  <inertial>
+    <!-- <origin rpy="0 -1.0471975512 0" xyz="0 0 0" /> -->
+    <origin rpy="0 -0.785398163 0" xyz="0 0 0" />
+    <mass value="${lidarMass}" />
+    <xacro:cylinder_inertia m="${lidarMass}" r="${lidarRadius}" h="${lidarHeight}"/>
+  </inertial>
+  <visual>
+    <!-- <origin rpy="0 0.785398163 0" xyz="0 0 0"/> -->
+    <geometry>
+      <cylinder length="0.041" radius="0.038" />
+    </geometry>
+    <material name="silver"/>
+  </visual>
+  <collision>
+    <!-- <origin rpy="0 0.785398163 0" xyz="0 0 0"/> -->
+    <geometry>
+      <cylinder length="0.041" radius="0.038" />
+    </geometry>
+  </collision>
+</link>
 <joint name="right_front_rev" type="continuous">
   <origin rpy="0 0 0" xyz="0.254 -0.254 0.101276"/>
@@ -148,4 +172,9 @@
   <axis xyz="0.0 1.0 0.0"/>
 </joint>
+<joint name="baselink_lidar" type="fixed">
+  <origin rpy="0 0.785398163 0" xyz="0.275 -0.3 0.4" />
+  <parent link="base_link" />
+  <child link="lidar" />
+</joint>
 <xacro:include filename="$(find realsense_ros_gazebo)/xacro/depthcam.xacro"/>
 <xacro:realsense_d435 sensor_name="d435_forward" parent_link="base_link" rate="10">

File: lunabot_sim/lunabot_description/urdf/lunabot.xacro (robot description, xacro)
@@ -1,164 +1,195 @@
 <?xml version="1.0" ?>
 <robot name="lunabot" xmlns:xacro="http://www.ros.org/wiki/xacro">
-<xacro:property name="PI" value="3.1415926535897931"/>
-<xacro:property name="chassisHeight" value="0.2"/>
-<xacro:property name="chassisLength" value="0.82"/>
-<xacro:property name="chassisWidth" value="0.5"/>
-<xacro:property name="chassisMass" value="55"/>
-<xacro:property name="wheelWidth" value="0.05"/>
-<xacro:property name="wheelRadius" value="0.15"/>
-<xacro:property name="wheelMass" value="5"/>
-<xacro:macro name="box_inertia" params="m x y z">
-  <inertia  ixx="${m*(y*y+z*z)/12}" ixy = "0" ixz = "0"
-    iyy="${m*(x*x+z*z)/12}" iyz = "0"
-    izz="${m*(x*x+z*z)/12}"
-  />
-</xacro:macro>
-<xacro:macro name="cylinder_inertia" params="m r h">
-  <inertia  ixx="${m*(3*r*r+h*h)/12}" ixy = "0" ixz = "0"
-    iyy="${m*(3*r*r+h*h)/12}" iyz = "0"
-    izz="${m*r*r/2}"
-  />
-</xacro:macro>
-<xacro:include filename="$(find lunabot_description)/urdf/materials.xacro" />
-<link name="base_link"/>
-<link name="chassis">
-  <visual>
-    <origin rpy="0 0 0" xyz="0 0 0.215"/>
-    <geometry>
-      <mesh filename="package://lunabot_description/meshes/base_link.stl" scale="0.001 0.001 0.001"/>
-    </geometry>
-    <material name="silver"/>
-  </visual>
-  <collision>
+  <xacro:property name="PI" value="3.1415926535897931"/>
+  <xacro:property name="chassisHeight" value="0.2"/>
+  <xacro:property name="chassisLength" value="0.82"/>
+  <xacro:property name="chassisWidth" value="0.5"/>
+  <xacro:property name="chassisMass" value="55" />
+  <xacro:property name="wheelWidth" value="0.05"/>
+  <xacro:property name="wheelRadius" value="0.15"/>
+  <xacro:property name="wheelMass" value="5"/>
+  <xacro:property name="lidarMass" value="0.190" />
+  <xacro:property name="lidarRadius" value="0.038" />
+  <xacro:property name="lidarHeight" value="0.041" />
+  <xacro:macro name="box_inertia" params="m x y z">
+    <inertia  ixx="${m*(y*y+z*z)/12}" ixy = "0" ixz = "0"
+      iyy="${m*(x*x+z*z)/12}" iyz = "0"
+      izz="${m*(x*x+z*z)/12}"
+    />
+  </xacro:macro>
+  <xacro:macro name="cylinder_inertia" params="m r h">
+    <inertia  ixx="${m*(3*r*r+h*h)/12}" ixy = "0" ixz = "0"
+      iyy="${m*(3*r*r+h*h)/12}" iyz = "0"
+      izz="${m*r*r/2}"
+    />
+  </xacro:macro>
+  <xacro:include filename="$(find lunabot_description)/urdf/materials.xacro" />
+  <!-- LINKS ================= -->
+  <link name="base_link"/>
+  <link name="chassis">
+    <visual>
+      <origin rpy="0 0 0" xyz="0 0 0.215"/>
+      <geometry>
+        <mesh filename="package://lunabot_description/meshes/base_link.stl" scale="0.001 0.001 0.001"/>
+      </geometry>
+      <material name="silver"/>
+    </visual>
+    <collision>
+      <origin rpy="0 0 0" xyz="0 0 0"/>
+      <geometry>
+        <mesh filename="package://lunabot_description/meshes/base_link.stl" scale="0.001 0.001 0.001"/>
+      </geometry>
+    </collision>
+  </link>
+  <link name="right_front">
+    <inertial>
+      <origin rpy="0 0 0" xyz="0 0 0"/>
+      <mass value="${wheelMass}"/>
+      <xacro:cylinder_inertia m="${wheelMass}" r="${wheelRadius}" h="${wheelWidth}"/>
+    </inertial>
+    <visual>
+      <origin rpy="0 0 0" xyz="-0.275 0.3 0"/>
+      <geometry>
+        <mesh filename="package://lunabot_description/meshes/right_front.stl" scale="0.001 0.001 0.001"/>
+      </geometry>
+      <material name="silver"/>
+    </visual>
+    <collision>
+      <origin rpy="0 0 0" xyz="-0.275 0.3 0"/>
+      <geometry>
+        <mesh filename="package://lunabot_description/meshes/right_front.stl" scale="0.001 0.001 0.001"/>
+      </geometry>
+    </collision>
+  </link>
+  <link name="left_front">
+    <inertial>
+      <origin rpy="0 0 0" xyz="0 0 0"/>
+      <mass value="${wheelMass}"/>
+      <xacro:cylinder_inertia m="${wheelMass}" r="${wheelRadius}" h="${wheelWidth}"/>
+    </inertial>
+    <visual>
+      <origin rpy="0 0 0" xyz="-0.275 -0.3 0"/>
+      <geometry>
+        <mesh filename="package://lunabot_description/meshes/left_front.stl" scale="0.001 0.001 0.001"/>
+      </geometry>
+      <material name="silver"/>
+    </visual>
+    <collision>
+      <origin rpy="0 0 0" xyz="-0.275 -0.3 0"/>
+      <geometry>
+        <mesh filename="package://lunabot_description/meshes/left_front.stl" scale="0.001 0.001 0.001"/>
+      </geometry>
+    </collision>
+  </link>
+  <link name="left_back">
+    <inertial>
+      <origin rpy="0 0 0" xyz="0 0 0"/>
+      <mass value="${wheelMass}"/>
+      <xacro:cylinder_inertia m="${wheelMass}" r="${wheelRadius}" h="${wheelWidth}"/>
+    </inertial>
+    <visual>
+      <origin rpy="0 0 0" xyz="0.275 -0.3 0"/>
+      <geometry>
+        <mesh filename="package://lunabot_description/meshes/left_back.stl" scale="0.001 0.001 0.001"/>
+      </geometry>
+      <material name="silver"/>
+    </visual>
+    <collision>
+      <origin rpy="0 0 0" xyz="0.275 -0.3 0"/>
+      <geometry>
+        <mesh filename="package://lunabot_description/meshes/left_back.stl" scale="0.001 0.001 0.001"/>
+      </geometry>
+    </collision>
+  </link>
+  <link name="right_back">
+    <inertial>
+      <origin rpy="0 0 0" xyz="0 0 0"/>
+      <mass value="${wheelMass}"/>
+      <xacro:cylinder_inertia m="${wheelMass}" r="${wheelRadius}" h="${wheelWidth}"/>
+    </inertial>
+    <visual>
+      <origin rpy="0 0 0" xyz="0.275 0.3 0"/>
+      <geometry>
+        <mesh filename="package://lunabot_description/meshes/right_back.stl" scale="0.001 0.001 0.001"/>
+      </geometry>
+      <material name="silver"/>
+    </visual>
+    <collision>
+      <origin rpy="0 0 0" xyz="0.275 0.3 0"/>
+      <geometry>
+        <mesh filename="package://lunabot_description/meshes/right_back.stl" scale="0.001 0.001 0.001"/>
+      </geometry>
+    </collision>
+  </link>
+  <link name="lidar">
+    <inertial>
+      <!-- <origin rpy="0 -1.0471975512 0" xyz="0 0 0" /> -->
+      <origin rpy="0 -0.785398163 0" xyz="0 0 0" />
+      <mass value="${lidarMass}" />
+      <xacro:cylinder_inertia m="${lidarMass}" r="${lidarRadius}" h="${lidarHeight}"/>
+    </inertial>
+    <visual>
+      <!-- <origin rpy="0 0.785398163 0" xyz="0 0 0"/> -->
+      <geometry>
+        <cylinder length="0.041" radius="0.038" />
+      </geometry>
+      <material name="silver"/>
+    </visual>
+    <collision>
+      <!-- <origin rpy="0 0.785398163 0" xyz="0 0 0"/> -->
+      <geometry>
+        <cylinder length="0.041" radius="0.038" />
+      </geometry>
+    </collision>
+  </link>
+  <link name="usb_cam_link"/>
+  <!-- JOINTS ====================== -->
+  <joint name="base_link" type="fixed">
     <origin rpy="0 0 0" xyz="0 0 0"/>
-    <geometry>
-      <mesh filename="package://lunabot_description/meshes/base_link.stl" scale="0.001 0.001 0.001"/>
-    </geometry>
-  </collision>
-</link>
-<link name="right_front">
-  <inertial>
-    <origin rpy="0 0 0" xyz="0 0 0"/>
-    <mass value="${wheelMass}"/>
-    <xacro:cylinder_inertia m="${wheelMass}" r="${wheelRadius}" h="${wheelWidth}"/>
-  </inertial>
-  <visual>
-    <origin rpy="0 0 0" xyz="-0.275 0.3 0"/>
-    <geometry>
-      <mesh filename="package://lunabot_description/meshes/right_front.stl" scale="0.001 0.001 0.001"/>
-    </geometry>
-    <material name="silver"/>
-  </visual>
-  <collision>
-    <origin rpy="0 0 0" xyz="-0.275 0.3 0"/>
-    <geometry>
-      <mesh filename="package://lunabot_description/meshes/right_front.stl" scale="0.001 0.001 0.001"/>
-    </geometry>
-  </collision>
-</link>
-<link name="left_front">
-  <inertial>
-    <origin rpy="0 0 0" xyz="0 0 0"/>
-    <mass value="${wheelMass}"/>
-    <xacro:cylinder_inertia m="${wheelMass}" r="${wheelRadius}" h="${wheelWidth}"/>
-  </inertial>
-  <visual>
-    <origin rpy="0 0 0" xyz="-0.275 -0.3 0"/>
-    <geometry>
-      <mesh filename="package://lunabot_description/meshes/left_front.stl" scale="0.001 0.001 0.001"/>
-    </geometry>
-    <material name="silver"/>
-  </visual>
-  <collision>
-    <origin rpy="0 0 0" xyz="-0.275 -0.3 0"/>
-    <geometry>
-      <mesh filename="package://lunabot_description/meshes/left_front.stl" scale="0.001 0.001 0.001"/>
-    </geometry>
-  </collision>
-</link>
-<link name="left_back">
-  <inertial>
-    <origin rpy="0 0 0" xyz="0 0 0"/>
-    <mass value="${wheelMass}"/>
-    <xacro:cylinder_inertia m="${wheelMass}" r="${wheelRadius}" h="${wheelWidth}"/>
-  </inertial>
-  <visual>
-    <origin rpy="0 0 0" xyz="0.275 -0.3 0"/>
-    <geometry>
-      <mesh filename="package://lunabot_description/meshes/left_back.stl" scale="0.001 0.001 0.001"/>
-    </geometry>
-    <material name="silver"/>
-  </visual>
-  <collision>
-    <origin rpy="0 0 0" xyz="0.275 -0.3 0"/>
-    <geometry>
-      <mesh filename="package://lunabot_description/meshes/left_back.stl" scale="0.001 0.001 0.001"/>
-    </geometry>
-  </collision>
-</link>
-<link name="right_back">
-  <inertial>
-    <origin rpy="0 0 0" xyz="0 0 0"/>
-    <mass value="${wheelMass}"/>
-    <xacro:cylinder_inertia m="${wheelMass}" r="${wheelRadius}" h="${wheelWidth}"/>
-  </inertial>
-  <visual>
-    <origin rpy="0 0 0" xyz="0.275 0.3 0"/>
-    <geometry>
-      <mesh filename="package://lunabot_description/meshes/right_back.stl" scale="0.001 0.001 0.001"/>
-    </geometry>
-    <material name="silver"/>
-  </visual>
-  <collision>
-    <origin rpy="0 0 0" xyz="0.275 0.3 0"/>
-    <geometry>
-      <mesh filename="package://lunabot_description/meshes/right_back.stl" scale="0.001 0.001 0.001"/>
-    </geometry>
-  </collision>
-</link>
-<joint name="base_link" type="fixed">
-  <origin rpy="0 0 0" xyz="0 0 0"/>
-  <parent link="base_link"/>
-  <child link="chassis"/>
-  <axis xyz="0.0 1.0 0.0"/>
-</joint>
-<joint name="right_front_rev" type="continuous">
-  <origin rpy="0 0 0" xyz="0.275 -0.3 0.14"/>
-  <parent link="chassis"/>
-  <child link="right_front"/>
-  <axis xyz="0.0 1.0 0.0"/>
-</joint>
-<joint name="left_front_rev" type="continuous">
-  <origin rpy="0 0 0" xyz="0.275 0.3 0.14"/>
-  <parent link="chassis"/>
-  <child link="left_front"/>
-  <axis xyz="0.0 -1.0 0.0"/>
-</joint>
-<joint name="left_back_rev" type="continuous">
-  <origin rpy="0 0 0" xyz="-0.275 0.3 0.14"/>
-  <parent link="chassis"/>
-  <child link="left_back"/>
-  <axis xyz="0.0 -1.0 0.0"/>
-</joint>
-<joint name="right_back_rev" type="continuous">
-  <origin rpy="0 0 0" xyz="-0.275 -0.3 0.14"/>
-  <parent link="chassis"/>
-  <child link="right_back"/>
-  <axis xyz="0.0 1.0 0.0"/>
-</joint>
-<link name="d455_back_link"/>
-<joint name="depth_cam_jnt" type="fixed">
-    <origin rpy="0 0 0" xyz="0.405 -0.10 0.45"/>
-  <parent link="base_link"/>
-  <child link="d455_back_link"/>
-  <axis xyz="0.0 1.0 0.0"/>
-</joint>
-<link name="usb_cam_link"/>
-<joint name="usb_cam_jnt" type="fixed">
-    <origin rpy="0 1.57 3.14" xyz="-0.405 0.10 0.65"/>
-  <parent link="base_link"/>
-  <child link="usb_cam_link"/>
-  <axis xyz="0.0 1.0 0.0"/>
-</joint>
+    <parent link="base_link"/>
+    <child link="chassis"/>
+    <axis xyz="0.0 1.0 0.0"/>
+  </joint>
+  <joint name="right_front_rev" type="continuous">
+    <origin rpy="0 0 0" xyz="0.275 -0.3 0.14"/>
+    <parent link="chassis"/>
+    <child link="right_front"/>
+    <axis xyz="0.0 1.0 0.0"/>
+  </joint>
+  <joint name="left_front_rev" type="continuous">
+    <origin rpy="0 0 0" xyz="0.275 0.3 0.14"/>
+    <parent link="chassis"/>
+    <child link="left_front"/>
+    <axis xyz="0.0 -1.0 0.0"/>
+  </joint>
+  <joint name="left_back_rev" type="continuous">
+    <origin rpy="0 0 0" xyz="-0.275 0.3 0.14"/>
+    <parent link="chassis"/>
+    <child link="left_back"/>
+    <axis xyz="0.0 -1.0 0.0"/>
+  </joint>
+  <joint name="right_back_rev" type="continuous">
+    <origin rpy="0 0 0" xyz="-0.275 -0.3 0.14"/>
+    <parent link="chassis"/>
+    <child link="right_back"/>
+    <axis xyz="0.0 1.0 0.0"/>
+  </joint>
+  <link name="d455_back_link"/>
+  <joint name="depth_cam_jnt" type="fixed">
+      <origin rpy="0 0 0" xyz="0.405 -0.10 0.45"/>
+    <parent link="base_link"/>
+    <child link="d455_back_link"/>
+    <axis xyz="0.0 1.0 0.0"/>
+  </joint>
+  <joint name="usb_cam_jnt" type="fixed">
+      <origin rpy="0 1.57 3.14" xyz="-0.405 0.10 0.65"/>
+    <parent link="base_link"/>
+    <child link="usb_cam_link"/>
+    <axis xyz="0.0 1.0 0.0"/>
+  </joint>
+  <joint name="baselink_lidar" type="fixed">
+    <origin rpy="0 0.785398163 0" xyz="0.275 -0.3 0.4" />
+    <parent link="base_link" />
+    <child link="lidar" />
+  </joint>
 </robot>
